File: schematics/Embedded-Systems-Class-Project/Embedded-Systems-Class-Project.kicad_sch (KiCad schematic)
At the start: 14 parts

Commit message: Issue 21 - opisanie komunikacji bluetooth
Parts:
- added U?: BMD-330_BT_Module_(simplified_pinout), symbol Embedded-Systems-Class-Project:BMD-330_BT_Module_(simplified_pinout)
Connections:
- net +3.3V: now also U?. (VCC)
- net GND: now also U?. (VCC)
- net OUT: now also U?. (VCC)
- net at U?.2 (SCL), U?.A3 (PB8): now also U?. (VCC)
Changed lines of the file:
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@@
   (junction (at 222.25 40.64) (diameter 0) (color 0 0 0 0)
   )
+  (junction (at 83.82 86.36) (diameter 0) (color 0 0 0 0)
+  )
   (junction (at 158.75 67.31) (diameter 0) (color 0 0 0 0)
+  )
+  (junction (at 86.36 83.82) (diameter 0) (color 0 0 0 0)
   )
   (no_connect (at 88.9 72.39))
@@
     (stroke (width 0) (type default) (color 0 0 0 0))
   )
+  (wire (pts (xy 86.36 83.82) (xy 74.93 83.82))
+    (stroke (width 0) (type default) (color 0 0 0 0))
+  )
   (wire (pts (xy 190.5 67.31) (xy 195.58 67.31))
     (stroke (width 0) (type default) (color 0 0 0 0))
@@
     (stroke (width 0) (type default) (color 0 0 0 0))
   )
+  (wire (pts (xy 83.82 86.36) (xy 91.44 86.36))
+    (stroke (width 0) (type default) (color 0 0 0 0))
+  )
   (wire (pts (xy 248.92 125.73) (xy 250.19 125.73))
     (stroke (width 0) (type default) (color 0 0 0 0))
   )
+  (wire (pts (xy 86.36 107.95) (xy 113.03 107.95))
+    (stroke (width 0) (type default) (color 0 0 0 0))
+  )
   (wire (pts (xy 222.25 66.04) (xy 222.25 67.31))
     (stroke (width 0) (type default) (color 0 0 0 0))
@@
     (stroke (width 0) (type default) (color 0 0 0 0))
   )
+  (wire (pts (xy 102.87 105.41) (xy 113.03 105.41))
+    (stroke (width 0) (type default) (color 0 0 0 0))
+  )
   (wire (pts (xy 222.25 40.64) (xy 240.03 40.64))
     (stroke (width 0) (type default) (color 0 0 0 0))
@@
     (stroke (width 0) (type default) (color 0 0 0 0))
   )
+  (wire (pts (xy 83.82 86.36) (xy 83.82 110.49))
+    (stroke (width 0) (type default) (color 0 0 0 0))
+  )
   (wire (pts (xy 158.75 40.64) (xy 158.75 44.45))
     (stroke (width 0) (type default) (color 0 0 0 0))
@@
     (stroke (width 0) (type default) (color 0 0 0 0))
   )
+  (wire (pts (xy 86.36 83.82) (xy 86.36 107.95))
+    (stroke (width 0) (type default) (color 0 0 0 0))
+  )
   (wire (pts (xy 180.34 81.28) (xy 143.51 81.28))
     (stroke (width 0) (type default) (color 0 0 0 0))
@@
     (stroke (width 0) (type default) (color 0 0 0 0))
   )
-  (wire (pts (xy 74.93 86.36) (xy 91.44 86.36))
+  (wire (pts (xy 74.93 86.36) (xy 83.82 86.36))
     (stroke (width 0) (type default) (color 0 0 0 0))
   )
@@
     (stroke (width 0) (type default) (color 0 0 0 0))
   )
+  (wire (pts (xy 83.82 110.49) (xy 113.03 110.49))
+    (stroke (width 0) (type default) (color 0 0 0 0))
+  )
   (wire (pts (xy 158.75 67.31) (xy 158.75 69.85))
     (stroke (width 0) (type default) (color 0 0 0 0))
@@
     (stroke (width 0) (type default) (color 0 0 0 0))
   )
+  (wire (pts (xy 102.87 102.87) (xy 113.03 102.87))
+    (stroke (width 0) (type default) (color 0 0 0 0))
+  )
   (wire (pts (xy 91.44 86.36) (xy 104.14 86.36))
     (stroke (width 0) (type default) (color 0 0 0 0))
@@
     (stroke (width 0) (type default) (color 0 0 0 0))
   )
-  (wire (pts (xy 88.9 83.82) (xy 74.93 83.82))
+  (wire (pts (xy 88.9 83.82) (xy 86.36 83.82))
     (stroke (width 0) (type default) (color 0 0 0 0))
   )
@@
     (pin "9")
   )
+  (symbol (lib_id "Embedded-Systems-Class-Project:BMD-330_BT_Module_(simplified_pinout)") (at 124.46 106.68 0) (unit 1)
+    (in_bom yes) (on_board yes)
+    (property "Reference" "U?" (id 0) (at 123.19 116.84 0)
+      (effects (font (size 1.27 1.27)) (justify left))
+    )
+    (property "Value" "BMD-330_BT_Module_(simplified_pinout)" (id 1) (at 105.41 114.3 0)
+      (effects (font (size 1.27 1.27)) (justify left))
+    )
+    (property "Footprint" "" (id 2) (at 124.46 106.68 0)
+      (effects (font (size 1.27 1.27)) hide)
+    )
+    (property "Datasheet" "" (id 3) (at 124.46 106.68 0)
+      (effects (font (size 1.27 1.27)) hide)
+    )
+    (pin "")
+    (pin "")
+    (pin "")
+    (pin "")
+  )
   (symbol (lib_id "power:GND") (at 190.5 69.85 0) (unit 1)
     (in_bom yes) (on_board yes) (fields_autoplaced)
@@
     )
     (property "Datasheet" "" (id 3) (at 222.25 35.56 0)
+      (effects (font (size 1.27 1.27)) hide)
+    )
+    (pin "1")
+  )
+  (symbol (lib_id "power:+3.3V") (at 102.87 102.87 90) (unit 1)
+    (in_bom yes) (on_board yes)
+    (property "Reference" "#PWR?" (id 0) (at 106.68 102.87 0)
+      (effects (font (size 1.27 1.27)) hide)
+    )
+    (property "Value" "+3.3V" (id 1) (at 93.98 102.87 90)
+      (effects (font (size 1.27 1.27)) (justify right))
+    )
+    (property "Footprint" "" (id 2) (at 102.87 102.87 0)
+      (effects (font (size 1.27 1.27)) hide)
+    )
+    (property "Datasheet" "" (id 3) (at 102.87 102.87 0)
       (effects (font (size 1.27 1.27)) hide)
     )
@@
     (pin "9")
   )
+  (symbol (lib_id "power:GND") (at 102.87 105.41 270) (unit 1)
+    (in_bom yes) (on_board yes)
+    (property "Reference" "#PWR?" (id 0) (at 96.52 105.41 0)
+      (effects (font (size 1.27 1.27)) hide)
+    )
+    (property "Value" "GND" (id 1) (at 95.25 105.41 90)
+      (effects (font (size 1.27 1.27)) (justify left))
+    )
+    (property "Footprint" "" (id 2) (at 102.87 105.41 0)
+      (effects (font (size 1.27 1.27)) hide)
+    )
+    (property "Datasheet" "" (id 3) (at 102.87 105.41 0)
+      (effects (font (size 1.27 1.27)) hide)
+    )
+    (pin "1")
+  )
   (symbol (lib_id "Device:C") (at 199.39 67.31 270) (unit 1)
     (in_bom yes) (on_board yes) (fields_autoplaced)
@@
       (reference "#PWR?") (unit 1) (value "+3.3V") (footprint "")
     )
+    (path "/ba68e46a-b18d-4ba6-a00e-034f5a11fbb0"
+      (reference "#PWR?") (unit 1) (value "+3.3V") (footprint "")
+    )
     (path "/d0f0e08b-133c-44a1-946f-551add08edad"
       (reference "#PWR?") (unit 1) (value "GND") (footprint "")
@@
       (reference "#PWR?") (unit 1) (value "GND") (footprint "")
     )
+    (path "/e7a1cd1a-c056-4775-a041-a5243a99a735"
+      (reference "#PWR?") (unit 1) (value "GND") (footprint "")
+    )
     (path "/f1dcfb07-bcfe-4f3d-9507-6c63394d8b8a"
       (reference "#PWR?") (unit 1) (value "GND") (footprint "")
@@
       (reference "U?") (unit 1) (value "LCD_16X2") (footprint "")
     )
+    (path "/70310f65-ed20-4441-aa7b-23d94e08d9b6"
+      (reference "U?") (unit 1) (value "BMD-330_BT_Module_(simplified_pinout)") (footprint "")
+    )
     (path "/a7737520-3a3a-4c82-8c7a-5d4c51d46684"

Commit message: feat(#27): Realizacja issue nr. #27
Parts:
- added SW? (x4): SW_MEC_5G, symbol Switch:SW_MEC_5G
- added U?: Buzzer_Module, symbol Embedded-Systems-Class-Project:Buzzer_Module
Connections:
- net GND: now also SW?.3 (B), SW?.3 (B), SW?.3 (B), SW?.3 (B), SW?.4 (B), SW?.4 (B), SW?.4 (B), SW?.4 (B), U?. (VCC)
- net at U?.H12 (PD13): now also SW?.1 (A), SW?.2 (A)
- net at U?.J12 (PD10): now also SW?.1 (A), SW?.2 (A)
- net at U?.K12 (PB13): now also SW?.1 (A), SW?.2 (A)
- net at U?.K4 (PA5): now also U?. (VCC)
- net at U?.L12 (PB12): now also SW?.1 (A), SW?.2 (A)
- new net +5V: U?. (VCC)
Other:
- moved on the sheet: U?
