File: schematics/Embedded-Systems-Class-Project/Embedded-Systems-Class-Project.kicad_sch (KiCad schematic)
At the start: 20 parts

Commit message: Realizacja issue 21 - przechowywanie danyc
Connections:
- net +3.3V: now also U?.4 (VDD)
- net GND: now also U?.6 (VSS)
- net at U?.B10 (PC12): now also U?.5 (CLK)
- net at U?.B11 (PC10): now also U?.1 (DAT2)
- net at U?.C10 (PC11): now also U?.2 (CD/DAT3)
- net at U?.C8 (PD2): now also U?.3 (CMD)
- net at U?.D12 (PC9): now also U?.8 (DAT1)
- net at U?.E10 (PC8): now also U?.7 (DAT0)
Other:
- moved on the sheet: C?, TC?, U?

Commit message: Update Embedded-Systems-Class-Project.kicad_sch
Connections:
- net +3.3V: now also U?. (VCC)
- net GND: now also U?. (VCC)
- net OUT: now also U?. (VCC)
- net at U?. (VCC), U?.2 (SCL), U?.A3 (PB8): now also U?. (VCC)
Other:
- moved on the sheet: U?
